File: EAGLE/project/main_board.sch (EAGLE design)
At the start: 14 parts

Commit message: update main board
Parts:
- added LXDC1: LXDC55, LXDC55:LXDC55
- added X1: MKDSN1,5/3-5,08, con-phoenix-508:MKDSN1,5/3-5,08
Connections:
- net N$1 renamed CE
- net N$3 renamed SCK
- net N$4 renamed MOSI
- net N$5 renamed MISO
- net ULTRA_SONIC_1 renamed ECHO
- net ULTRA_SONIC_2 renamed TRIG
- removed net N$2: NRF24L1.CSN, RASPBERRY_PI.GPIO26
- new net 5V_LXDC55: LXDC1.OUTPUT, SERVO_1.2, SERVO_2.2, SERVO_3.2
- new net BATTERY+: LXDC1.INPUT, X1-1.KL, X1-2.KL
- new net CSN: NRF24L1.CSN, RASPBERRY_PI.GPIO8/!SPI_CE0!
- net 5V: no longer SERVO_1.1, SERVO_2.1, SERVO_3.1
- net GND: now also LXDC1.GND, SERVO_1.1, SERVO_2.1, SERVO_3.1, X1-3.KL; no longer SERVO_1.2, SERVO_2.2, SERVO_3.2

Commit message: update main board
Connections:
- removed net CE: NRF24L1.CE, RASPBERRY_PI.GPIO19
- removed net PWM_SERVO_1: RASPBERRY_PI.GPIO5, SERVO_1.3
- removed net PWM_SERVO_2: RASPBERRY_PI.GPIO6, SERVO_2.3
- removed net PWM_SERVO_3: RASPBERRY_PI.GPIO13, SERVO_3.3
- new net NRF_CE_GPIO5: NRF24L1.CE, RASPBERRY_PI.GPIO5
- new net SERVO1_GPIO13: RASPBERRY_PI.GPIO13, SERVO_1.3
- new net SERVO2_GPIO12: RASPBERRY_PI.GPIO12, SERVO_2.3
- new net SERVO3_GPIO19: RASPBERRY_PI.GPIO19, SERVO_3.3
Changed lines of the file:
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@@
-</segment>
-</net>
-<net name="PWM_SERVO_1" class="0">
-<segment>
-<pinref part="RASPBERRY_PI" gate="G$1" pin="GPIO5"/>
-<wire x1="25.4" y1="12.7" x2="58.42" y2="12.7" width="0.1524" layer="91"/>
-<wire x1="58.42" y1="12.7" x2="58.42" y2="-7.62" width="0.1524" layer="91"/>
-<pinref part="SERVO_1" gate="A" pin="3"/>
-<wire x1="96.52" y1="-7.62" x2="58.42" y2="-7.62" width="0.1524" layer="91"/>
-</segment>
-</net>
-<net name="PWM_SERVO_2" class="0">
-<segment>
-<pinref part="RASPBERRY_PI" gate="G$1" pin="GPIO6"/>
-<wire x1="25.4" y1="10.16" x2="55.88" y2="10.16" width="0.1524" layer="91"/>
-<pinref part="SERVO_2" gate="A" pin="3"/>
-<wire x1="55.88" y1="10.16" x2="55.88" y2="-25.4" width="0.1524" layer="91"/>
-<wire x1="55.88" y1="-25.4" x2="96.52" y2="-25.4" width="0.1524" layer="91"/>
-</segment>
-</net>
-<net name="PWM_SERVO_3" class="0">
-<segment>
-<pinref part="RASPBERRY_PI" gate="G$1" pin="GPIO13"/>
-<wire x1="25.4" y1="5.08" x2="53.34" y2="5.08" width="0.1524" layer="91"/>
-<pinref part="SERVO_3" gate="A" pin="3"/>
-<wire x1="53.34" y1="5.08" x2="53.34" y2="-43.18" width="0.1524" layer="91"/>
-<wire x1="53.34" y1="-43.18" x2="96.52" y2="-43.18" width="0.1524" layer="91"/>
 </segment>
 </net>
@@
 <pinref part="GPS" gate="A" pin="3"/>
 <wire x1="35.56" y1="-71.12" x2="96.52" y2="-71.12" width="0.1524" layer="91"/>
-</segment>
-</net>
-<net name="CE" class="0">
-<segment>
-<pinref part="RASPBERRY_PI" gate="G$1" pin="GPIO19"/>
-<wire x1="25.4" y1="0" x2="68.58" y2="0" width="0.1524" layer="91"/>
-<wire x1="68.58" y1="0" x2="68.58" y2="-55.88" width="0.1524" layer="91"/>
-<wire x1="68.58" y1="-55.88" x2="-20.32" y2="-55.88" width="0.1524" layer="91"/>
-<pinref part="NRF24L1" gate="G$1" pin="CE"/>
-<wire x1="-20.32" y1="-55.88" x2="-20.32" y2="-109.22" width="0.1524" layer="91"/>
-<wire x1="-20.32" y1="-109.22" x2="-17.78" y2="-109.22" width="0.1524" layer="91"/>
 </segment>
 </net>
@@
 </segment>
 </net>
+<net name="SERVO1_GPIO13" class="0">
+<segment>
+<pinref part="RASPBERRY_PI" gate="G$1" pin="GPIO13"/>
+<wire x1="25.4" y1="5.08" x2="78.74" y2="5.08" width="0.1524" layer="91"/>
+<wire x1="78.74" y1="5.08" x2="78.74" y2="-7.62" width="0.1524" layer="91"/>
+<pinref part="SERVO_1" gate="A" pin="3"/>
+<wire x1="78.74" y1="-7.62" x2="96.52" y2="-7.62" width="0.1524" layer="91"/>
+</segment>
+</net>
+<net name="SERVO2_GPIO12" class="0">
+<segment>
+<pinref part="RASPBERRY_PI" gate="G$1" pin="GPIO12"/>
+<wire x1="25.4" y1="7.62" x2="76.2" y2="7.62" width="0.1524" layer="91"/>
+<wire x1="76.2" y1="7.62" x2="76.2" y2="-25.4" width="0.1524" layer="91"/>
+<pinref part="SERVO_2" gate="A" pin="3"/>
+<wire x1="76.2" y1="-25.4" x2="96.52" y2="-25.4" width="0.1524" layer="91"/>
+</segment>
+</net>
+<net name="SERVO3_GPIO19" class="0">
+<segment>
+<pinref part="RASPBERRY_PI" gate="G$1" pin="GPIO19"/>
+<wire x1="25.4" y1="0" x2="73.66" y2="0" width="0.1524" layer="91"/>
+<pinref part="SERVO_3" gate="A" pin="3"/>
+<wire x1="73.66" y1="0" x2="73.66" y2="-43.18" width="0.1524" layer="91"/>
+<wire x1="73.66" y1="-43.18" x2="96.52" y2="-43.18" width="0.1524" layer="91"/>
+</segment>
+</net>
+<net name="NRF_CE_GPIO5" class="0">
+<segment>
+<pinref part="RASPBERRY_PI" gate="G$1" pin="GPIO5"/>
+<wire x1="25.4" y1="12.7" x2="53.34" y2="12.7" width="0.1524" layer="91"/>
+<wire x1="53.34" y1="12.7" x2="53.34" y2="-86.36" width="0.1524" layer="91"/>
+<wire x1="53.34" y1="-86.36" x2="-33.02" y2="-86.36" width="0.1524" layer="91"/>
+<pinref part="NRF24L1" gate="G$1" pin="CE"/>
+<wire x1="-33.02" y1="-86.36" x2="-33.02" y2="-109.22" width="0.1524" layer="91"/>
+<wire x1="-33.02" y1="-109.22" x2="-17.78" y2="-109.22" width="0.1524" layer="91"/>
+</segment>
+</net>
